File: eagle/schematic.brd (EAGLE design)
At the start: 100 x 80 mm, 4 parts, among them U1 SN74HC595N

Commit message: PCB update
Parts:
- added 100N_1: (no value), rcl:C025-025X050
- added 100N_2, 100N_3, CAP1, CAP2: (no value), rcl:C050-025X075
- added C1: (no value), rcl:E2,5-5
- added CLOCK_B, CS_B, GND, GND1_B, GND2_B, MISC1, MISC2, MISC3, MISC4, MISC5, OUTPUT, RCK_B, RESET_ARD, RESET_OUT, RESET_OUT_2, RESET_SID, RW_B, RX1_B, SCK_B, SER_B, TX0_B, VCC, VDD: LSP11, solpad:LSP11
- moved R1 12.5 mm to (73.7, 62.2), turned to 90 degrees
- moved U$2 11.7 mm to (58.4, 52.1)
- moved U1 10.8 mm to (76.2, 41.9)
- moved U$1 8.52 mm to (16.5, 64.8)
Connections:
- removed net GND: U1.8
- removed net VCC: U$1.21, U1.16
- new net 0: 100N_1.2, 100N_2.1, 100N_3.1, GND.MP, R1.1, U$1.23, U$2.14, U1.13, U1.8
- new net N$18: 100N_3.2, U$2.28, VDD.MP
- new net N$19: 100N_1.1, 100N_2.2, RESET_OUT.MP, RESET_OUT_2.MP, U$1.21, U$2.25, U1.10, U1.16, VCC.MP
- new net N$20: CAP2.1, U$2.4
- new net N$21: RESET_SID.MP, U$2.5
- new net N$22: C1.-, OUTPUT.MP
- new net N$23: CAP2.2, U$2.3
- new net N$24: CAP1.2, U$2.1
- new net N$25: CAP1.1, U$2.2
- new net N$26: SER_B.MP, U$1.5, U1.14
- new net N$27: SCK_B.MP, U$1.7, U1.11
- new net N$28: RCK_B.MP, U$1.6, U1.12
- new net N$29: MISC2.MP, U$1.8
- new net N$30: MISC1.MP, U$1.9
- new net N$31: RESET_ARD.MP, U$1.22
- new net N$32: MISC3.MP, U$1.16
- new net N$33: MISC4.MP, U$1.15
- new net N$34: MISC5.MP, U$1.14
- new net N$35: TX0_B.MP, U$1.1
- new net N$36: RX1_B.MP, U$1.2
- new net N$37: GND1_B.MP, U$1.3
- new net N$38: GND2_B.MP, U$1.4
- net N$14: now also CS_B.MP
- net N$15: now also RW_B.MP
- net N$16: now also CLOCK_B.MP
- net N$17: now also C1.+, R1.2; no longer R1.1
Routing:
- net 0: track 0.00 -> 209.3 mm
- net N$26: track 0.00 -> 164.7 mm
- net N$28: track 0.00 -> 144.9 mm
- net N$19: track 0.00 -> 138.6 mm
- net N$27: track 0.00 -> 126.5 mm
- net N$16: track 0.00 -> 89.5 mm
- net N$15: track 0.00 -> 78.9 mm
- net N$14: track 0.00 -> 70.2 mm
- net N$5: track 0.00 -> 21.7 mm
- net N$4: track 0.00 -> 21.7 mm
- net N$3: track 0.00 -> 21.7 mm
- net N$2: track 0.00 -> 21.7 mm
- net N$18: track 0.00 -> 20.3 mm
- net N$1: track 0.00 -> 19.6 mm
- net N$13: track 0.00 -> 17.6 mm
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